Commit message: added in front_axle_controller

File: src/robot_description/urdf/gazebo_essentials_base.xacro (robot description, xacro)
@@ -35,6 +35,6 @@
 <!-- front axle controller -->
 <Gazebo>
-  <plugin name="joint_state_publisher" filename="libgazebo_ros_joint_state_publisher.so">
-  <jointName>front_axle_joint</jointName>
+  <plugin name="gazebo_ros_control" filename="libgazebo_ros_control.so">
+    <robotParam>/robot_description</robotParam>
   </plugin>
 </Gazebo>

File: src/robot_description/urdf/robot_essentials.xacro (robot description, xacro)
@@ -118,9 +118,9 @@
   <type>transmission_interface/SimpleTransmission</type>
   <actuator name="front_motor">
-    <hardwareInterface>hardware_interface/PositionJointInterface</hardwareInterface>
+    <hardwareInterface>hardware_interface/EffortJointInterface</hardwareInterface>
     <mechanicalReduction>1</mechanicalReduction>
   </actuator>
-  <joint name="front_joint">
-    <hardwareInterface>hardware_interface/PositionJointInterface</hardwareInterface>
+  <joint name="front_axle_joint">
+    <hardwareInterface>hardware_interface/EffortJointInterface</hardwareInterface>
   </joint>
 </transmission>

Commit message: added in files for software/control to edit

File: src/robot_description/urdf/gazebo_essentials_base.xacro (robot description, xacro)
@@ -49,3 +49,45 @@
 </gazebo>
 </xacro:macro>
+<!--############################# Camera Vision #########################################-->
+<xacro:macro name="camera_vision">
+ <gazebo reference="camera_link">
+    <sensor type="camera" name="camera1">
+      <update_rate>30.0</update_rate>
+      <camera name="head">
+        <horizontal_fov>1.3962634</horizontal_fov>
+        <image>
+          <width>800</width>
+          <height>800</height>
+          <format>R8G8B8</format>
+        </image>
+        <clip>
+          <near>0.02</near>
+          <far>300</far>
+        </clip>
+        <noise>
+          <type>gaussian</type>
+          <!-- Noise is sampled independently per pixel on each frame.
+               That pixel's noise value is added to each of its color
+               channels, which at that point lie in the range [0,1]. -->
+          <mean>0.0</mean>
+          <stddev>0.007</stddev>
+        </noise>
+      </camera>
+      <plugin name="camera_controller" filename="libgazebo_ros_camera.so">
+        <alwaysOn>true</alwaysOn>
+        <updateRate>0.0</updateRate>
+        <cameraName>agbot/camera1</cameraName>
+        <imageTopicName>image_raw</imageTopicName>
+        <cameraInfoTopicName>camera_info</cameraInfoTopicName>
+        <frameName>camera_link</frameName>
+        <hackBaseline>0.07</hackBaseline>
+        <distortionK1>0.0</distortionK1>
+        <distortionK2>0.0</distortionK2>
+        <distortionK3>0.0</distortionK3>
+        <distortionT1>0.0</distortionT1>
+        <distortionT2>0.0</distortionT2>
+      </plugin>
+    </sensor>
+  </gazebo>
+</xacro:macro>
 </robot>

File: src/robot_description/urdf/robot_base.urdf.xacro (robot description, xacro)
@@ -61,3 +61,7 @@
 <xacro:wheel_friction prefix="rear_left"/>
 <xacro:wheel_friction prefix="rear_right"/>
+<!-- camera joint -->
+<xacro:camera_join/>
+<xacro:camera/>
+<xacro:camera_vision/>
 </robot>

File: src/robot_description/urdf/robot_essentials.xacro (robot description, xacro)
@@ -1,4 +1,5 @@
 <?xml version="1.0"?>
 <robot xmlns:xacro="http://ros.org/wiki/xacro" name="robot_essentials" >
+<xacro:property name="camera_link" value="0.05" /> <!-- Size of square 'camera' box -->
 <!-- defining wheels -->
 <xacro:macro name="robot_wheel" params="prefix">
@@ -126,3 +127,35 @@
 </transmission>
 </xacro:macro>
+<!-- define camera joint -->
+<xacro:macro name="camera_join">
+  <joint name="camera_joint" type="fixed">
+    <axis xyz="0 1 0" />
+    <origin xyz=".4 0 .05" rpy="0 0 0"/>
+    <parent link="base_link"/>
+    <child link="camera_link"/>
+  </joint>
+</xacro:macro>
+<xacro:macro name="camera">
+  <!-- Camera -->
+  <link name="camera_link">
+    <collision>
+      <origin xyz="0 0 0" rpy="0 0 0"/>
+      <geometry>
+    <box size="${camera_link} ${camera_link} ${camera_link}"/>
+      </geometry>
+    </collision>
+    <visual>
+      <origin xyz="0 0 0" rpy="0 0 0"/>
+      <geometry>
+    <box size="${camera_link} ${camera_link} ${camera_link}"/>
+      </geometry>
+      <material name=""/>
+    </visual>
+    <inertial>
+      <mass value="1e-5" />
+      <origin xyz="0 0 0" rpy="0 0 0"/>
+      <inertia ixx="1e-6" ixy="0" ixz="0" iyy="1e-6" iyz="0" izz="1e-6" />
+    </inertial>
+  </link>
+</xacro:macro>
 </robot>
